File: _autosave-prominny_kicad.kicad_pcb (KiCad board)
At the start: 2 copper layers, 134.2 x 105.8 mm, 35 parts, among them J1 Conn_01x08_Female, SW1 SW_Push, SW2 SW_Push, SW3 SW_Push, SW4 SW_Push, SW5 SW_Push, SW6 SW_Push, SW7 SW_Push, U1 TRRS, U2 ProMicro

Commit message: arranges, added edgecuts, started routing
Parts:
- removed J1: Conn_01x08_Female, Connector_PinHeader_1.00mm:PinHeader_1x08_P1.00mm_Vertical
- R1, R2: moved to B.Cu
- moved D6 84.7 mm to (220.6, 57.1)
- moved D7 71.9 mm to (234.9, 60.3)
- moved D8 56.4 mm to (246.7, 86.2)
- moved D5 56.4 mm to (201.6, 52.4)
- moved D9 46.1 mm to (246.8, 106.4)
- moved D4 38.2 mm to (182.6, 57.1)
- moved D10 37.0 mm to (233.3, 140.5)
- moved D3 21.7 mm to (163.5, 68.3)
- moved R1 7.38 mm to (146.7, 126.2), turned to 0 degrees
- moved R2 4.15 mm to (151.6, 126.2), turned to 0 degrees
- turned D1 to 0 degrees
- turned D2 to 0 degrees
- renumbered D9 to D10, D4 to D3, D6 to D4, D8 to D5, D10 to D6, D3 to D7, D5 to D8, D7 to D9
Connections:
- net leddata1 renamed Net-(D6-Pad2)
- D13 pad 1: Net-(D13-Pad1) -> power
- D14 pad 1: Net-(D14-Pad1) -> power
Routing:
- net ground: track 185.6 -> 375.9 mm
- net power: track 0.00 -> 138.9 mm
- net col4: track 0.00 -> 130.4 mm
- net col3: track 0.00 -> 120.0 mm
- net col2: track 0.00 -> 103.2 mm
- net sda: track 0.00 -> 100.1 mm, vias 0 -> 1
- net scl: track 0.00 -> 94.5 mm, vias 0 -> 1
- net col1: track 0.00 -> 94.5 mm
- net col0: track 0.00 -> 63.6 mm
- net row0: track 266.9 -> 297.2 mm
- net leds: track 9.92 -> 32.2 mm
- net Net-(D1-Pad2): track 0.00 -> 21.1 mm
- net connection: track 0.00 -> 17.0 mm
- net A1: track 0.00 -> 14.4 mm
- net reset: track 0.00 -> 14.4 mm
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